Commit message: arakno class finally working

File: arakno/resources/urdfs/arakno.urdf (robot description, URDF)
Before this commit: robot arakno, 13 links, 12 joints
Joints:
- joint BL_lowerleg_joint: limit lower=0.05 upper=1.08 effort=30 velocity=5 -> lower=0.05 upper=1.08 effort=300 velocity=5
- joint BL_shoulder_joint: limit lower=-0.785 upper=0.785 effort=30 velocity=5 -> lower=-0.785 upper=0.785 effort=300 velocity=5
- joint BL_upperleg_joint: limit lower=-0.785 upper=0.785 effort=30 velocity=5 -> lower=-0.785 upper=0.785 effort=300 velocity=5
- joint BR_lowerleg_joint: limit lower=0.05 upper=1.08 effort=30 velocity=5 -> lower=0.05 upper=1.08 effort=300 velocity=5
- joint BR_shoulder_joint: limit lower=-0.785 upper=0.785 effort=30 velocity=5 -> lower=-0.785 upper=0.785 effort=300 velocity=5
- joint BR_upperleg_joint: limit lower=-0.785 upper=0.785 effort=30 velocity=5 -> lower=-0.785 upper=0.785 effort=300 velocity=5
- joint FL_lowerleg_joint: limit lower=0.05 upper=1.08 effort=30 velocity=5 -> lower=0.05 upper=1.08 effort=300 velocity=5
- joint FL_shoulder_joint: limit lower=-0.785 upper=0.785 effort=30 velocity=5 -> lower=-0.785 upper=0.785 effort=300 velocity=5
- joint FL_upperleg_joint: limit lower=-0.785 upper=0.785 effort=30 velocity=5 -> lower=-0.785 upper=0.785 effort=300 velocity=5
- joint FR_lowerleg_joint: limit lower=0.05 upper=1.08 effort=30 velocity=5 -> lower=0.05 upper=1.08 effort=300 velocity=5
- joint FR_shoulder_joint: limit lower=-0.785 upper=0.785 effort=30 velocity=5 -> lower=-0.785 upper=0.785 effort=300 velocity=5
- joint FR_upperleg_joint: limit lower=-0.785 upper=0.785 effort=30 velocity=5 -> lower=-0.785 upper=0.785 effort=300 velocity=5
